Commit message: renaming + reorienting axes in urdf

File: urdf/protobot_core.xacro (robot description, xacro)
@@ -5,26 +5,27 @@
   <!-- Constants for robot dimensions -->
   <xacro:property name="PI" value="3.1415926535897931"/>
-  <xacro:property name="base_mass" value="0.5" /> <!-- arbitrary value for base mass -->
-  <xacro:property name="base_width" value="0.2" />
-  <xacro:property name="base_length" value="0.2" />
-  <xacro:property name="base_height" value="0.05" />
+  <xacro:property name="chassis_mass" value="0.5" /> <!-- arbitrary value for base mass -->
+  <xacro:property name="chassis_length" value="0.3" />
+  <xacro:property name="chassis_width" value="0.25" />
+  <xacro:property name="chassis_height" value="0.15" />
+  <xacro:property name="wheel_base" value="0.31" /> <!-- make this bigger than chassis_width -->
   <xacro:property name="wheel_mass" value="0.3" /> <!-- arbitrary value for wheel mass -->
-  <xacro:property name="wheel_len" value="0.010" />
-  <xacro:property name="wheel_radius" value="0.03" />
+  <xacro:property name="wheel_width" value="0.030" />
+  <xacro:property name="wheel_radius" value="0.05" />
+  <xacro:property name="wheel_axis_vertical_offset" value="-0.04" /> <!-- signed distance from chassis center to wheel axis -->
   <xacro:property name="caster_wheel_mass" value="0.1" /> <!-- arbitrary value for caster wheel mass -->
-  <xacro:property name="caster_wheel_radius" value="0.015" />
-  <xacro:property name="z_offset" value="-${base_height/4}" /> <!-- Space btw top of beam and the each joint -->
-  <!-- Base Link -->
-  <link name="${prefix}body_link">
+  <xacro:property name="caster_wheel_radius" value="${-wheel_axis_vertical_offset + wheel_radius - chassis_height/2}" />
+  <!-- Chassis Link -->
+  <link name="${prefix}chassis_link">
     <collision>
       <origin xyz="0 0 0" rpy="0 0 0"/>
       <geometry>
-        <box size="${base_width} ${base_length} ${base_height}"/>
+        <box size="${chassis_length} ${chassis_width} ${chassis_height}"/>
       </geometry>
     </collision>
     <visual>
-      <origin xyz="0 0 ${base_height/2}" rpy="0 0 0"/>
+      <origin xyz="0 0 0" rpy="0 0 0"/>
       <geometry>
-        <box size="${base_width} ${base_length} ${base_height}"/>
+        <box size="${chassis_length} ${chassis_width} ${chassis_height}"/>
       </geometry>
       <material name="orange"/>
@@ -32,87 +33,89 @@
     <inertial>
       <origin xyz="0 0 0" rpy="0 0 0"/>
-      <mass value="${base_mass}"/>
+      <mass value="${chassis_mass}"/>
       <inertia
-        ixx="${base_mass / 12.0 * (base_length*base_length + base_height*base_height)}" ixy="0.0" ixz="0.0"
-        iyy="${base_mass / 12.0 * (base_height*base_height + base_width*base_width)}" iyz="0.0"
-        izz="${base_mass / 12.0 * (base_width*base_width + base_length*base_length)}"/>
+        ixx="${chassis_mass / 12.0 * (chassis_width*chassis_width + chassis_height*chassis_height)}" ixy="0.0" ixz="0.0"
+        iyy="${chassis_mass / 12.0 * (chassis_height*chassis_height + chassis_length*chassis_length)}" iyz="0.0"
+        izz="${chassis_mass / 12.0 * (chassis_length*chassis_length + chassis_width*chassis_width)}"/>
       </inertial>
     </link>
     <joint name="${prefix}base_to_body" type="fixed">
       <parent link="${parent}"/>
-      <child link="${prefix}body_link"/>
+      <child link="${prefix}chassis_link"/>
       <xacro:insert_block name="origin"/>
     </joint>
     <joint name="${prefix}left_wheel_joint" type="continuous">
-      <parent link="${prefix}body_link"/>
+      <parent link="${prefix}chassis_link"/>
       <child link="${prefix}left_wheel"/>
-      <origin xyz="0 -${base_width/2} ${z_offset}" rpy="0 0 0"/>
-      <axis xyz="0 1 0"/>
-      <dynamics damping="0.2"/>
-      <limit effort="100" velocity="1.0"/>
+      <origin xyz="0 ${chassis_length/2} ${wheel_axis_vertical_offset}" rpy="${-PI/2} 0 0"/>
+      <axis xyz="0 0 1"/>
+      <!-- <dynamics damping="0.2"/>
+      <limit effort="100" velocity="1.0"/> -->
     </joint>
     <!-- left wheel Link -->
     <link name="${prefix}left_wheel">
       <collision>
-        <origin xyz="0 0 0" rpy="${PI/2} 0 0"/>
+        <origin xyz="0 0 0" rpy="0 0 0"/>
         <geometry>
-          <cylinder length="${wheel_len}" radius="${wheel_radius}"/>
+          <!-- Sphere has point-contact with the ground, which makes simulation more stable -->
+          <sphere radius="${wheel_radius}"/>
         </geometry>
       </collision>
       <visual>
-        <origin xyz="0 0 0" rpy="${PI/2} 0 0"/>
+        <origin xyz="0 0 0" rpy="0 0 0"/>
         <geometry>
-          <cylinder length="${wheel_len}" radius="${wheel_radius}"/>
+          <cylinder length="${wheel_width}" radius="${wheel_radius}"/>
         </geometry>
         <material name="black"/>
       </visual>
       <inertial>
-        <origin xyz="0 0 0" rpy="${PI/2} 0 0"/>
+        <origin xyz="0 0 0" rpy="0 0 0"/>
         <mass value="${wheel_mass}"/>
         <inertia
-          ixx="${wheel_mass / 12.0 * (3*wheel_radius*wheel_radius + wheel_len*wheel_len)}" ixy="0.0" ixz="0.0"
-          iyy="${wheel_mass / 12.0 * (3*wheel_radius*wheel_radius + wheel_len*wheel_len)}" iyz="0.0"
+          ixx="${wheel_mass / 12.0 * (3*wheel_radius*wheel_radius + wheel_width*wheel_width)}" ixy="0.0" ixz="0.0"
+          iyy="${wheel_mass / 12.0 * (3*wheel_radius*wheel_radius + wheel_width*wheel_width)}" iyz="0.0"
           izz="${wheel_mass / 2.0 * wheel_radius*wheel_radius}"/>
         </inertial>
       </link>
     <joint name="${prefix}right_wheel_joint" type="continuous">
-      <parent link="${prefix}body_link"/>
+      <parent link="${prefix}chassis_link"/>
       <child link="${prefix}right_wheel"/>
-      <origin xyz="0 ${base_width/2} ${z_offset}" rpy="0 0 0"/>
-      <axis xyz="0 1 0"/>
-      <dynamics damping="0.2"/>
-      <limit effort="100" velocity="1.0"/>
+      <origin xyz="0 ${-chassis_length/2} ${wheel_axis_vertical_offset}" rpy="${PI/2} 0 0"/>
+      <axis xyz="0 0 1"/>
+      <!-- <dynamics damping="0.2"/>
+      <limit effort="100" velocity="1.0"/> -->
     </joint>
     <!-- right wheel Link -->
     <link name="${prefix}right_wheel">
       <collision>
-        <origin xyz="0 0 0" rpy="${PI/2} 0 0"/>
+        <origin xyz="0 0 0" rpy="0 0 0"/>
         <geometry>
-          <cylinder length="${wheel_len}" radius="${wheel_radius}"/>
+          <!-- Sphere has point-contact with the ground, which makes simulation more stable -->
+          <sphere radius="${wheel_radius}"/>
         </geometry>
       </collision>
       <visual>
-        <origin xyz="0 0 0" rpy="${PI/2} 0 0"/>
+        <origin xyz="0 0 0" rpy="0 0 0"/>
         <geometry>
-          <cylinder length="${wheel_len}" radius="${wheel_radius}"/>
+          <cylinder length="${wheel_width}" radius="${wheel_radius}"/>
         </geometry>
         <material name="black"/>
       </visual>
       <inertial>
-        <origin xyz="0 0 0" rpy="${PI/2} 0 0"/>
+        <origin xyz="0 0 0" rpy="0 0 0"/>
         <mass value="${wheel_mass}"/>
         <inertia
-          ixx="${wheel_mass / 12.0 * (3*wheel_radius*wheel_radius + wheel_len*wheel_len)}" ixy="0.0" ixz="0.0"
-          iyy="${wheel_mass / 12.0 * (3*wheel_radius*wheel_radius + wheel_len*wheel_len)}" iyz="0.0"
+          ixx="${wheel_mass / 12.0 * (3*wheel_radius*wheel_radius + wheel_width*wheel_width)}" ixy="0.0" ixz="0.0"
+          iyy="${wheel_mass / 12.0 * (3*wheel_radius*wheel_radius + wheel_width*wheel_width)}" iyz="0.0"
           izz="${wheel_mass / 2.0 * wheel_radius*wheel_radius}"/>
         </inertial>
       </link>
-    <joint name="${prefix}caster_frontal_wheel_joint" type="fixed">
-      <parent link="${prefix}body_link"/>
-      <child link="${prefix}caster_frontal_wheel"/>
-      <origin xyz="${base_width/2 - caster_wheel_radius} 0 ${z_offset}" rpy="0 0 0"/>
+    <joint name="${prefix}front_caster_wheel_joint" type="fixed">
+      <parent link="${prefix}chassis_link"/>
+      <child link="${prefix}front_caster_wheel"/>
+      <origin xyz="${chassis_length/2 - caster_wheel_radius} 0 ${-chassis_height/2}" rpy="0 0 0"/>
     </joint>
-    <!-- caster frontal wheel Link -->
-    <link name="${prefix}caster_frontal_wheel">
+    <!-- caster front wheel Link -->
+    <link name="${prefix}front_caster_wheel">
       <collision>
         <origin xyz="0 0 0" rpy="0 0 0"/>
@@ -137,11 +140,11 @@
         </inertial>
       </link>
-    <joint name="${prefix}caster_rear_wheel_joint" type="fixed">
-      <parent link="${prefix}body_link"/>
-      <child link="${prefix}caster_rear_wheel"/>
-      <origin xyz="${-base_width/2 + caster_wheel_radius} 0 ${z_offset}" rpy="0 0 0"/>
+    <joint name="${prefix}rear_caster_wheel_joint" type="fixed">
+      <parent link="${prefix}chassis_link"/>
+      <child link="${prefix}rear_caster_wheel"/>
+      <origin xyz="${-chassis_length/2 + caster_wheel_radius} 0 ${-chassis_height/2}" rpy="0 0 0"/>
     </joint>
     <!-- caster rear wheel Link -->
-    <link name="${prefix}caster_rear_wheel">
+    <link name="${prefix}rear_caster_wheel">
       <collision>
         <origin xyz="0 0 0" rpy="0 0 0"/>
@@ -168,7 +171,7 @@
     <!-- Hat joint -->
     <joint name="${prefix}hat_joint" type="fixed">
-      <parent link="${prefix}body_link"/>
+      <parent link="${prefix}chassis_link"/>
       <child link="${prefix}hat_link"/>
-      <origin xyz="0 0 ${base_height/2 + 0.02}" rpy="0 0 0"/>
+      <origin xyz="0 0 ${chassis_height/2}" rpy="0 0 0"/>
     </joint>
     <!-- Hat link -->

Commit message: FIxed right wheel axis to be opposite the left

File: urdf/protobot_core.xacro (robot description, xacro)
@@ -82,5 +82,5 @@
       <child link="${prefix}right_wheel"/>
       <origin xyz="0 ${-chassis_length/2} ${wheel_axis_vertical_offset}" rpy="${PI/2} 0 0"/>
-      <axis xyz="0 0 1"/>
+      <axis xyz="0 0 -1"/> <!-- Note that "Forward" rotation is opposite compared to the left wheel -->
       <!-- <dynamics damping="0.2"/>
       <limit effort="100" velocity="1.0"/> -->
