Commit message: adding gazebo and ros2 control xacro files

File: urdf/protobot.xacro (robot description, xacro)
@@ -4,6 +4,4 @@
     <xacro:arg name="prefix" default="" />
     <xacro:arg name="use_gazebo" default="false" />
-    <!-- TODO: What is mock hardware? -->
-    <xacro:arg name="use_mock_hardware" default="false" />
     <!-- Import different pieces of the protobot -->
     <!-- RVIZ colors -->
@@ -18,10 +16,10 @@
     </xacro:protobot_core>
     <!-- ROS2 Control -->
-    <!-- <xacro:include filename="$(find protobot_description)/urdf/protobot_control.xacro" />
-    <xacro:protobot_control name="protobot" prefix="$(arg prefix)" use_gazebo="$(arg use_gazebo)" /> -->
+    <xacro:include filename="$(find protobot_description)/urdf/protobot_control.xacro" />
+    <xacro:protobot_ros2_control name="protobot" prefix="$(arg prefix)" use_gazebo="$(arg use_gazebo)" />
     <!-- Gazebo-specific URDF -->
-    <!-- <xacro:if value="$(arg use_gazebo)">
+    <xacro:if value="$(arg use_gazebo)">
         <xacro:include filename="$(find protobot_description)/urdf/protobot_gazebo.xacro" />
         <xacro:protobot_gazebo prefix="$(arg prefix)"/>
-    </xacro:if> -->
+    </xacro:if>
 </robot>

File: urdf/protobot_control.xacro (robot description, xacro)
@@ -2,8 +2,8 @@
 <robot xmlns:xacro="http://www.ros.org/wiki/xacro">
   <!-- Define a macro that can be used to define the ros2 control interfaces -->
-  <xacro:macro name="protobot_control" params="name prefix use_gazebo:=^|false">
+  <xacro:macro name="protobot_ros2_control" params="name prefix use_gazebo:=^|false">
     <ros2_control name="${name}" type="system">
       <hardware>
-            <xacro:unless value="${use_mock_hardware}">
+            <!-- <xacro:unless value="${use_mock_hardware}">
           <plugin>ros2_control_demo_example_2/DiffBotSystemHardware</plugin>
           <param name="example_param_hw_start_duration_sec">0</param>
@@ -13,5 +13,5 @@
           <plugin>mock_components/GenericSystem</plugin>
           <param name="calculate_dynamics">true</param>
-      </xacro:if>
+      </xacro:if> -->
         <xacro:if value="${use_gazebo}">
           <plugin>gz_ros2_control/GazeboSimSystem</plugin>
@@ -19,17 +19,23 @@
         <xacro:unless value="${use_gazebo}">
           <!-- TODO: Add the protobot_steering_controller plugin here -->
-          <plugin>ros2_control_demo_example_9/RRBotSystemPositionOnlyHardware</plugin>
+          <!-- <plugin>ros2_control_demo_example_9/RRBotSystemPositionOnlyHardware</plugin>
           <param name="example_param_hw_start_duration_sec">0</param>
           <param name="example_param_hw_stop_duration_sec">3.0</param>
-          <param name="example_param_hw_slowdown">100</param>
+          <param name="example_param_hw_slowdown">100</param> -->
         </xacro:unless>
       </hardware>
       <joint name="${prefix}left_wheel_joint">
-        <command_interface name="velocity"/>
+        <command_interface name="velocity">
+          <param name="min">-10</param>
+          <param name="max">10</param>
+        </command_interface>
         <state_interface name="position"/>
         <state_interface name="velocity"/>
       </joint>
       <joint name="${prefix}right_wheel_joint">
-        <command_interface name="velocity"/>
+        <command_interface name="velocity">
+          <param name="min">-10</param>
+          <param name="max">10</param>
+        </command_interface>
         <state_interface name="position"/>
         <state_interface name="velocity"/>

File: urdf/protobot_core.xacro (robot description, xacro)
@@ -17,5 +17,5 @@
   <xacro:property name="caster_wheel_radius" value="${-wheel_axis_vertical_offset + wheel_radius - chassis_height/2}" />
   <!-- Chassis Link -->
-  <link name="${prefix}chassis_link">
+  <link name="${prefix}chassis">
     <collision>
       <origin xyz="0 0 0" rpy="0 0 0"/>
@@ -40,11 +40,11 @@
       </inertial>
     </link>
-    <joint name="${prefix}base_to_body" type="fixed">
+    <joint name="${prefix}base_to_chassis_joint" type="fixed">
       <parent link="${parent}"/>
-      <child link="${prefix}chassis_link"/>
+      <child link="${prefix}chassis"/>
       <xacro:insert_block name="origin"/>
     </joint>
     <joint name="${prefix}left_wheel_joint" type="continuous">
-      <parent link="${prefix}chassis_link"/>
+      <parent link="${prefix}chassis"/>
       <child link="${prefix}left_wheel"/>
       <origin xyz="0 ${chassis_length/2} ${wheel_axis_vertical_offset}" rpy="${-PI/2} 0 0"/>
@@ -79,5 +79,5 @@
       </link>
     <joint name="${prefix}right_wheel_joint" type="continuous">
-      <parent link="${prefix}chassis_link"/>
+      <parent link="${prefix}chassis"/>
       <child link="${prefix}right_wheel"/>
       <origin xyz="0 ${-chassis_length/2} ${wheel_axis_vertical_offset}" rpy="${PI/2} 0 0"/>
@@ -112,5 +112,5 @@
       </link>
     <joint name="${prefix}front_caster_wheel_joint" type="fixed">
-      <parent link="${prefix}chassis_link"/>
+      <parent link="${prefix}chassis"/>
       <child link="${prefix}front_caster_wheel"/>
       <origin xyz="${chassis_length/2 - caster_wheel_radius} 0 ${-chassis_height/2}" rpy="0 0 0"/>
@@ -141,5 +141,5 @@
       </link>
     <joint name="${prefix}rear_caster_wheel_joint" type="fixed">
-      <parent link="${prefix}chassis_link"/>
+      <parent link="${prefix}chassis"/>
       <child link="${prefix}rear_caster_wheel"/>
       <origin xyz="${-chassis_length/2 + caster_wheel_radius} 0 ${-chassis_height/2}" rpy="0 0 0"/>
@@ -171,10 +171,10 @@
     <!-- Hat joint -->
     <joint name="${prefix}hat_joint" type="fixed">
-      <parent link="${prefix}chassis_link"/>
-      <child link="${prefix}hat_link"/>
+      <parent link="${prefix}chassis"/>
+      <child link="${prefix}hat"/>
       <origin xyz="0 0 ${chassis_height/2}" rpy="0 0 0"/>
     </joint>
     <!-- Hat link -->
-    <link name="${prefix}hat_link">
+    <link name="${prefix}hat">
       <visual>
         <origin xyz="0 0 0" rpy="0 0 0"/>

Commit message: put base_link back in protobot_core

File: urdf/protobot.xacro (robot description, xacro)
@@ -7,12 +7,8 @@
     <!-- RVIZ colors -->
     <xacro:include filename="$(find protobot_description)/urdf/materials.xacro" />
-    <!-- Dummy link is used as root (for gazebo) -->
-    <link name="base_link"/>
     <!-- Use macros from imported files to define the full protobot -->
     <!-- Core URDF -->
     <xacro:include filename="$(find protobot_description)/urdf/protobot_core.xacro" />
-    <xacro:protobot_core parent="base_link" prefix="$(arg prefix)">
-        <origin xyz="0 0 0" rpy="0 0 0" />
-    </xacro:protobot_core>
+    <xacro:protobot_core prefix="$(arg prefix)"/>
     <!-- ROS2 Control -->
     <xacro:include filename="$(find protobot_description)/urdf/protobot_control.xacro" />

File: urdf/protobot_core.xacro (robot description, xacro)
@@ -2,5 +2,5 @@
 <robot xmlns:xacro="http://www.ros.org/wiki/xacro">
 <!-- Modified from: https://github.com/ros-controls/ros2_control_demos/blob/master/ros2_control_demo_description/diffbot/urdf/diffbot_description.urdf.xacro -->
-  <xacro:macro name="protobot_core" params="parent prefix *origin">
+  <xacro:macro name="protobot_core" params="prefix">
   <!-- Constants for robot dimensions -->
   <xacro:property name="PI" value="3.1415926535897931"/>
@@ -16,4 +16,6 @@
   <xacro:property name="caster_wheel_mass" value="0.1" /> <!-- arbitrary value for caster wheel mass -->
   <xacro:property name="caster_wheel_radius" value="${-wheel_axis_vertical_offset + wheel_radius - chassis_height/2}" />
+  <!-- Dummy link with no inertiais used as root (for gazebo) -->
+  <link name="base_link"/>
   <!-- Chassis Link -->
   <link name="${prefix}chassis">
@@ -41,7 +43,7 @@
     </link>
     <joint name="${prefix}base_to_chassis_joint" type="fixed">
-      <parent link="${parent}"/>
+      <parent link="base_link"/>
       <child link="${prefix}chassis"/>
-      <xacro:insert_block name="origin"/>
+      <origin xyz="0 0 0" rpy="0 0 0" />
     </joint>
     <joint name="${prefix}left_wheel_joint" type="continuous">

Commit message: Add camera: add camera.xacro and new rviz config file

File: urdf/protobot.xacro (robot description, xacro)
@@ -11,4 +11,9 @@
     <xacro:include filename="$(find protobot_description)/urdf/protobot_core.xacro" />
     <xacro:protobot_core prefix="$(arg prefix)"/>
+    <!-- Camera -->
+    <xacro:include filename="$(find protobot_description)/urdf/camera.xacro" />
+    <xacro:camera parent="chassis" prefix="$(arg prefix)">
+        <origin xyz="0.15 0 0" rpy="0 0 0" />
+    </xacro:camera>
     <!-- ROS2 Control -->
     <xacro:include filename="$(find protobot_description)/urdf/protobot_control.xacro" />
