Commit message: cleanup comments + aesthetics

File: urdf/protobot_control.xacro (robot description, xacro)
@@ -5,22 +5,9 @@
     <ros2_control name="${name}" type="system">
       <hardware>
-            <!-- <xacro:unless value="${use_mock_hardware}">
-          <plugin>ros2_control_demo_example_2/DiffBotSystemHardware</plugin>
-          <param name="example_param_hw_start_duration_sec">0</param>
-          <param name="example_param_hw_stop_duration_sec">3.0</param>
-      </xacro:unless>
-      <xacro:if value="${use_mock_hardware}">
-          <plugin>mock_components/GenericSystem</plugin>
-          <param name="calculate_dynamics">true</param>
-      </xacro:if> -->
         <xacro:if value="${use_gazebo}">
           <plugin>gz_ros2_control/GazeboSimSystem</plugin>
         </xacro:if>
         <xacro:unless value="${use_gazebo}">
-          <!-- TODO: Add the protobot_steering_controller plugin here -->
-          <!-- <plugin>ros2_control_demo_example_9/RRBotSystemPositionOnlyHardware</plugin>
-          <param name="example_param_hw_start_duration_sec">0</param>
-          <param name="example_param_hw_stop_duration_sec">3.0</param>
-          <param name="example_param_hw_slowdown">100</param> -->
+          <!-- TODO: Add the protobot_steering_controller plugin here (see ros2_control_demos/example_9)-->
         </xacro:unless>
       </hardware>

File: urdf/protobot_core.xacro (robot description, xacro)
@@ -175,5 +175,5 @@
       <parent link="${prefix}chassis"/>
       <child link="${prefix}hat"/>
-      <origin xyz="0 0 ${chassis_height/2}" rpy="0 0 0"/>
+      <origin xyz="0.03 0 ${chassis_height/2}" rpy="0 0 0"/>
     </joint>
     <!-- Hat link -->
