Commit message: Raise COM and remove velocity limits so the robot can tip over

File: urdf/protobot_control.urdf.xacro (robot description, xacro)
@@ -14,6 +14,7 @@
       <joint name="${prefix}left_wheel_joint">
         <command_interface name="velocity">
-          <param name="min">-10</param>
-          <param name="max">10</param>
+        <!-- Currently unlimited; set to something reasonable later-->
+          <!-- <param name="min">-10</param>
+          <param name="max">10</param> -->
         </command_interface>
         <state_interface name="position"/>
@@ -22,6 +23,7 @@
       <joint name="${prefix}right_wheel_joint">
         <command_interface name="velocity">
-          <param name="min">-10</param>
-          <param name="max">10</param>
+          <!-- Currently unlimited; set to something reasonable later-->
+          <!-- <param name="min">-10</param>
+          <param name="max">10</param> -->
         </command_interface>
         <state_interface name="position"/>

File: urdf/protobot_core.urdf.xacro (robot description, xacro)
@@ -23,5 +23,5 @@
     <xacro:property name="chassis_length" value="0.3" />
     <xacro:property name="chassis_width" value="0.25" />
-    <xacro:property name="chassis_height" value="0.15" />
+    <xacro:property name="chassis_height" value="0.3" />
     <xacro:property name="wheel_base" value="0.31" /> <!-- make this bigger than chassis_width -->
     <xacro:property name="wheel_mass" value="0.2" /> <!-- arbitrary value for wheel mass -->
