Commit message: removed gz_frame_id from sensors and removed color choice from IMU to avoid sdf errors (may need gz_frame_id later)

File: urdf/camera.urdf.xacro (robot description, xacro)
@@ -38,4 +38,5 @@
             <camera>
                 <camera_info_topic>/camera/camera_info</camera_info_topic>
+                <optical_frame_id>camera_link_optical</optical_frame_id>
                 <horizontal_fov>1.089</horizontal_fov>
                 <image>
@@ -50,5 +51,5 @@
             </camera>
             <topic>camera/image_raw</topic>
-            <gz_frame_id>camera_link_optical</gz_frame_id>
+            <!-- <gz_frame_id>camera_link_optical</gz_frame_id> -->
         </sensor>
     </gazebo>

File: urdf/imu_sensor.urdf.xacro (robot description, xacro)
@@ -13,9 +13,5 @@
         width:=0.03785
         height:=0.01338
-        material_name:='imu_black'
-        material_color:='0.1 0.1 0.1 1'
-        gazebo_material_ambient:='0.1 0.1 0.1 1'
-        gazebo_material_diffuse:='0.1 0.1 0.1 1'
-        gazebo_material_specular:='0.1 0.1 0.1 1'
+        material_name:='blue'
         update_rate:='15.0'
         topic_name:='imu/data'
@@ -30,7 +26,5 @@
                     <box size="${length} ${width} ${height}"/>
                 </geometry>
-                <material name="${material_name}">
-                    <color rgba="${material_color}"/>
-                </material>
+                <material name="${material_name}"/>
             </visual>
             <inertial>
@@ -52,9 +46,5 @@
         </joint>
         <gazebo reference="${prefix}imu_link">
-            <material>
-                <ambient>${gazebo_material_ambient}</ambient>
-                <diffuse>${gazebo_material_diffuse}</diffuse>
-                <specular>${gazebo_material_specular}</specular>
-            </material>
+            <material>Gazebo/Blue</material>
             <sensor name="${prefix}imu_sensor" type="imu">
                 <topic>${topic_name}</topic>
@@ -62,5 +52,5 @@
                 <always_on>${always_on}</always_on>
                 <visualize>${visualize}</visualize>
-                <gz_frame_id>${prefix}imu_link</gz_frame_id>
+                <!-- <gz_frame_id>${prefix}imu_link</gz_frame_id> -->
             </sensor>
         </gazebo>

Commit message: use_gazebo arg for camera and IMU

File: urdf/camera.urdf.xacro (robot description, xacro)
@@ -1,5 +1,5 @@
 <?xml version="1.0"?>
 <robot xmlns:xacro="http://www.ros.org/wiki/xacro" >
-  <xacro:macro name="camera" params="parent prefix *origin">
+  <xacro:macro name="camera" params="parent prefix *origin use_gazebo:=false">
     <joint name="camera_joint" type="fixed">
         <parent link="${parent}"/>
@@ -30,28 +30,30 @@
     </joint>
     <link name="${prefix}camera_link_optical"></link>
-    <gazebo reference="${prefix}camera_link">
-        <material>Gazebo/Red</material>
-        <sensor name="camera" type="camera">
-            <pose> 0 0 0 0 0 0 </pose>
-            <visualize>true</visualize>
-            <update_rate>10</update_rate>
-            <camera>
-                <camera_info_topic>/camera/camera_info</camera_info_topic>
-                <optical_frame_id>camera_link_optical</optical_frame_id>
-                <horizontal_fov>1.089</horizontal_fov>
-                <image>
-                    <format>R8G8B8</format>
-                    <width>640</width>
-                    <height>480</height>
-                </image>
-                <clip>
-                    <near>0.05</near>
-                    <far>8.0</far>
-                </clip>
-            </camera>
-            <topic>camera/image_raw</topic>
-            <!-- <gz_frame_id>camera_link_optical</gz_frame_id> -->
-        </sensor>
-    </gazebo>
+    <xacro:if value="${use_gazebo}">
+        <gazebo reference="${prefix}camera_link">
+            <material>Gazebo/Red</material>
+            <sensor name="camera" type="camera">
+                <pose> 0 0 0 0 0 0 </pose>
+                <visualize>true</visualize>
+                <update_rate>10</update_rate>
+                <camera>
+                    <camera_info_topic>/camera/camera_info</camera_info_topic>
+                    <optical_frame_id>camera_link_optical</optical_frame_id>
+                    <horizontal_fov>1.089</horizontal_fov>
+                    <image>
+                        <format>R8G8B8</format>
+                        <width>640</width>
+                        <height>480</height>
+                    </image>
+                    <clip>
+                        <near>0.05</near>
+                        <far>8.0</far>
+                    </clip>
+                </camera>
+                <topic>camera/image_raw</topic>
+                <!-- <gz_frame_id>camera_link_optical</gz_frame_id> -->
+            </sensor>
+        </gazebo>
+    </xacro:if>
   </xacro:macro>
 </robot>

File: urdf/imu_sensor.urdf.xacro (robot description, xacro)
@@ -19,4 +19,5 @@
         visualize:=false
         *origin
+        use_gazebo:=false
     ">
         <link name="${prefix}imu_link">
@@ -45,14 +46,16 @@
             <xacro:insert_block name="origin"/>
         </joint>
-        <gazebo reference="${prefix}imu_link">
-            <material>Gazebo/Blue</material>
-            <sensor name="${prefix}imu_sensor" type="imu">
-                <topic>${topic_name}</topic>
-                <update_rate>${update_rate}</update_rate>
-                <always_on>${always_on}</always_on>
-                <visualize>${visualize}</visualize>
-                <!-- <gz_frame_id>${prefix}imu_link</gz_frame_id> -->
-            </sensor>
-        </gazebo>
+        <xacro:if value="${use_gazebo}">
+            <gazebo reference="${prefix}imu_link">
+                <material>Gazebo/Blue</material>
+                <sensor name="${prefix}imu_sensor" type="imu">
+                    <topic>${topic_name}</topic>
+                    <update_rate>${update_rate}</update_rate>
+                    <always_on>${always_on}</always_on>
+                    <visualize>${visualize}</visualize>
+                    <!-- <gz_frame_id>${prefix}imu_link</gz_frame_id> -->
+                </sensor>
+            </gazebo>
+        </xacro:if>
     </xacro:macro>
 </robot>

File: urdf/protobot.urdf.xacro (robot description, xacro)
@@ -30,10 +30,10 @@
     <!-- Camera -->
     <xacro:include filename="$(find protobot_description)/urdf/camera.urdf.xacro" />
-    <xacro:camera parent="chassis" prefix="$(arg prefix)">
+    <xacro:camera parent="chassis" prefix="$(arg prefix)" use_gazebo="$(arg use_gazebo)">
         <origin xyz="${chassis_length} 0 0.1" rpy="0 0 0" />
     </xacro:camera>
     <!-- Inertial Measurement Unit (IMU) -->
     <xacro:include filename="$(find protobot_description)/urdf/imu_sensor.urdf.xacro" />
-    <xacro:imu_sensor prefix="$(arg prefix)" parent="chassis">
+    <xacro:imu_sensor prefix="$(arg prefix)" parent="chassis" use_gazebo="$(arg use_gazebo)">
         <origin xyz="${wheel_axis_horizontal_offset} 0 ${wheel_axis_vertical_offset}" rpy="0 0 0" />
     </xacro:imu_sensor>
