Commit message: Add imu: add imu_sensor.xacro

File: urdf/protobot.urdf.xacro (robot description, xacro)
@@ -16,4 +16,9 @@
         <origin xyz="0.15 0 0" rpy="0 0 0" />
     </xacro:camera>
+    <!-- Inertial Measurement Unit (IMU) -->
+    <xacro:include filename="$(find protobot_description)/urdf/imu_sensor.urdf.xacro" />
+    <xacro:imu_sensor prefix="$(arg prefix)" parent="chassis">
+        <origin xyz="0 0 0" rpy="0 0 0" />
+    </xacro:imu_sensor>
     <!-- ROS2 Control -->
     <xacro:include filename="$(find protobot_description)/urdf/protobot_control.urdf.xacro" />

Commit message: Use wheel_base + fix indentation + moved chassis origin to rear

File: urdf/protobot.urdf.xacro (robot description, xacro)
@@ -8,4 +8,5 @@
     <xacro:include filename="$(find protobot_description)/urdf/materials.urdf.xacro" />
     <!-- Use macros from imported files to define the full protobot -->
+    <!--TODO: Parametrize the core macro so that camera and IMU can be placed without hardcoding -->
     <!-- Core URDF -->
     <xacro:include filename="$(find protobot_description)/urdf/protobot_core.urdf.xacro" />
@@ -14,10 +15,10 @@
     <xacro:include filename="$(find protobot_description)/urdf/camera.urdf.xacro" />
     <xacro:camera parent="chassis" prefix="$(arg prefix)">
-        <origin xyz="0.15 0 0" rpy="0 0 0" />
+        <origin xyz="0.3 0 0.1" rpy="0 0 0" />
     </xacro:camera>
     <!-- Inertial Measurement Unit (IMU) -->
     <xacro:include filename="$(find protobot_description)/urdf/imu_sensor.urdf.xacro" />
     <xacro:imu_sensor prefix="$(arg prefix)" parent="chassis">
-        <origin xyz="0 0 0" rpy="0 0 0" />
+        <origin xyz="0.28 0 0.04" rpy="0 0 0" />
     </xacro:imu_sensor>
     <!-- ROS2 Control -->

File: urdf/protobot_core.urdf.xacro (robot description, xacro)
@@ -3,53 +3,68 @@
 <!-- Modified from: https://github.com/ros-controls/ros2_control_demos/blob/master/ros2_control_demo_description/diffbot/urdf/diffbot_description.urdf.xacro -->
   <xacro:macro name="protobot_core" params="prefix">
-  <!-- Constants for robot dimensions -->
-  <xacro:property name="PI" value="3.1415926535897931"/>
-  <xacro:property name="chassis_mass" value="1.0" /> <!-- arbitrary value for base mass -->
-  <xacro:property name="chassis_length" value="0.3" />
-  <xacro:property name="chassis_width" value="0.25" />
-  <xacro:property name="chassis_height" value="0.15" />
-  <xacro:property name="wheel_base" value="0.31" /> <!-- make this bigger than chassis_width -->
-  <xacro:property name="wheel_mass" value="0.2" /> <!-- arbitrary value for wheel mass -->
-  <xacro:property name="wheel_width" value="0.030" />
-  <xacro:property name="wheel_radius" value="0.06" />
-  <xacro:property name="wheel_axis_vertical_offset" value="-0.04" /> <!-- signed vertical distance from chassis center to wheel axis -->
-  <xacro:property  name="wheel_axis_horizontal_offset" value="${chassis_length/2 - 0.02}" /> <!-- signed horizontal distance from chassis center to wheel axis -->
-  <xacro:property name="caster_wheel_mass" value="0.1" /> <!-- arbitrary value for caster wheel mass -->
-  <xacro:property name="caster_wheel_radius" value="${-wheel_axis_vertical_offset + wheel_radius - chassis_height/2}" />
-  <!-- Dummy link with no inertiais used as root (for gazebo) -->
-  <link name="base_link"/>
-  <!-- Chassis Link -->
-  <link name="${prefix}chassis">
-    <collision>
-      <origin xyz="0 0 0" rpy="0 0 0"/>
-      <geometry>
-        <box size="${chassis_length} ${chassis_width} ${chassis_height}"/>
-      </geometry>
-    </collision>
-    <visual>
-      <origin xyz="0 0 0" rpy="0 0 0"/>
-      <geometry>
-        <box size="${chassis_length} ${chassis_width} ${chassis_height}"/>
-      </geometry>
-      <material name="orange"/>
-    </visual>
-    <inertial>
-      <origin xyz="0 0 0" rpy="0 0 0"/>
-      <mass value="${chassis_mass}"/>
-      <inertia
-        ixx="${chassis_mass / 12.0 * (chassis_width*chassis_width + chassis_height*chassis_height)}" ixy="0.0" ixz="0.0"
-        iyy="${chassis_mass / 12.0 * (chassis_height*chassis_height + chassis_length*chassis_length)}" iyz="0.0"
-        izz="${chassis_mass / 12.0 * (chassis_length*chassis_length + chassis_width*chassis_width)}"/>
-      </inertial>
+    <!-- TODO: Set these as macro parameters
+      prefix:=''
+      chassis_mass:='1.0'
+      chassis_length:='0.3'
+      chassis_width:='0.25'
+      chassis_height:='0.15'
+      wheel_base:='0.31'
+      wheel_mass:='0.2'
+      wheel_width:='0.030'
+      wheel_radius:='0.06'
+      wheel_axis_vertical_offset:='0.04'
+      wheel_axis_horizontal_offset:='0.28'
+      caster_wheel_radius:='0.02'
+      caster_wheel_mass:='0.1'
+  -->
+    <!-- Constants for robot dimensions -->
+    <xacro:property name="PI" value="3.1415926535897931"/>
+    <xacro:property name="chassis_mass" value="1.0" /> <!-- arbitrary value for base mass -->
+    <xacro:property name="chassis_length" value="0.3" />
+    <xacro:property name="chassis_width" value="0.25" />
+    <xacro:property name="chassis_height" value="0.15" />
+    <xacro:property name="wheel_base" value="0.31" /> <!-- make this bigger than chassis_width -->
+    <xacro:property name="wheel_mass" value="0.2" /> <!-- arbitrary value for wheel mass -->
+    <xacro:property name="wheel_width" value="0.030" />
+    <xacro:property name="wheel_radius" value="0.06" />
+    <xacro:property name="wheel_axis_vertical_offset" value="0.04" /> <!-- signed vertical distance from bottom of chassis to wheel axis -->
+    <xacro:property  name="wheel_axis_horizontal_offset" value="${chassis_length - 0.02}" /> <!-- signed horizontal distance from back of chassis to wheel axis -->
+    <xacro:property name="caster_wheel_mass" value="0.1" /> <!-- arbitrary value for caster wheel mass -->
+    <xacro:property name="caster_wheel_radius" value="${wheel_radius - wheel_axis_vertical_offset}" />
+    <!-- Dummy link with no inertiais used as root (for gazebo) -->
+    <link name="base_link"/>
+    <!-- Chassis Link -->
+    <link name="${prefix}chassis">
+      <collision>
+        <origin xyz="${chassis_length/2} 0 ${chassis_height/2}" rpy="0 0 0"/>
+        <geometry>
+          <box size="${chassis_length} ${chassis_width} ${chassis_height}"/>
+        </geometry>
+      </collision>
+      <visual>
+        <origin xyz="${chassis_length/2} 0 ${chassis_height/2}" rpy="0 0 0"/>
+        <geometry>
+          <box size="${chassis_length} ${chassis_width} ${chassis_height}"/>
+        </geometry>
+        <material name="orange"/>
+      </visual>
+      <inertial>
+        <origin xyz="${chassis_length/2} 0 ${chassis_height/2}" rpy="0 0 0"/>
+        <mass value="${chassis_mass}"/>
+        <inertia
+          ixx="${chassis_mass / 12.0 * (chassis_width*chassis_width + chassis_height*chassis_height)}" ixy="0.0" ixz="0.0"
+          iyy="${chassis_mass / 12.0 * (chassis_height*chassis_height + chassis_length*chassis_length)}" iyz="0.0"
+          izz="${chassis_mass / 12.0 * (chassis_length*chassis_length + chassis_width*chassis_width)}"/>
+        </inertial>
     </link>
     <joint name="${prefix}base_to_chassis_joint" type="fixed">
       <parent link="base_link"/>
       <child link="${prefix}chassis"/>
-      <origin xyz="0 0 0" rpy="0 0 0" />
+      <origin xyz="${-wheel_axis_horizontal_offset} 0 ${-wheel_axis_vertical_offset}" rpy="0 0 0" />
     </joint>
     <joint name="${prefix}left_wheel_joint" type="continuous">
       <parent link="${prefix}chassis"/>
       <child link="${prefix}left_wheel"/>
-      <origin xyz="${wheel_axis_horizontal_offset} ${chassis_length/2} ${wheel_axis_vertical_offset}" rpy="${-PI/2} 0 0"/>
+      <origin xyz="${wheel_axis_horizontal_offset} ${wheel_base/2} ${wheel_axis_vertical_offset}" rpy="${-PI/2} 0 0"/>
       <axis xyz="0 0 1"/>
       <!-- <dynamics damping="0.2"/>
@@ -79,10 +94,10 @@
           iyy="${wheel_mass / 12.0 * (3*wheel_radius*wheel_radius + wheel_width*wheel_width)}" iyz="0.0"
           izz="${wheel_mass / 2.0 * wheel_radius*wheel_radius}"/>
-        </inertial>
-      </link>
+      </inertial>
+    </link>
     <joint name="${prefix}right_wheel_joint" type="continuous">
       <parent link="${prefix}chassis"/>
       <child link="${prefix}right_wheel"/>
-      <origin xyz="${wheel_axis_horizontal_offset} ${-chassis_length/2} ${wheel_axis_vertical_offset}" rpy="${PI/2} 0 0"/>
+      <origin xyz="${wheel_axis_horizontal_offset} ${-wheel_base/2} ${wheel_axis_vertical_offset}" rpy="${PI/2} 0 0"/>
       <axis xyz="0 0 -1"/> <!-- Note that "Forward" rotation is opposite compared to the left wheel -->
       <!-- <dynamics damping="0.2"/>
@@ -112,39 +127,10 @@
           iyy="${wheel_mass / 12.0 * (3*wheel_radius*wheel_radius + wheel_width*wheel_width)}" iyz="0.0"
           izz="${wheel_mass / 2.0 * wheel_radius*wheel_radius}"/>
-        </inertial>
-      </link>
-    <!-- <joint name="${prefix}front_caster_wheel_joint" type="fixed">
-      <parent link="${prefix}chassis"/>
-      <child link="${prefix}front_caster_wheel"/>
-      <origin xyz="${chassis_length/2 - caster_wheel_radius} 0 ${-chassis_height/2}" rpy="0 0 0"/>
-    </joint> -->
-    <!-- caster front wheel Link -->
-    <!-- <link name="${prefix}front_caster_wheel">
-      <collision>
-        <origin xyz="0 0 0" rpy="0 0 0"/>
-        <geometry>
-          <sphere radius="${caster_wheel_radius}"/>
-        </geometry>
-      </collision>
-      <visual>
-        <origin xyz="0 0 0" rpy="0 0 0"/>
-        <geometry>
-          <sphere radius="${caster_wheel_radius}"/>
-        </geometry>
-        <material name="white"/>
-      </visual>
-      <inertial>
-        <origin xyz="0 0 0" rpy="0 0 0"/>
-        <mass value="${caster_wheel_mass}"/>
-        <inertia
-          ixx="${caster_wheel_mass * 0.4 * (caster_wheel_radius * caster_wheel_radius)}" ixy="0.0" ixz="0.0"
-          iyy="${caster_wheel_mass * 0.4 * (caster_wheel_radius * caster_wheel_radius)}" iyz="0.0"
-          izz="${caster_wheel_mass * 0.4 * (caster_wheel_radius * caster_wheel_radius)}"/>
-        </inertial>
-      </link> -->
+      </inertial>
+    </link>
     <joint name="${prefix}rear_caster_wheel_joint" type="fixed">
       <parent link="${prefix}chassis"/>
       <child link="${prefix}rear_caster_wheel"/>
-      <origin xyz="${-chassis_length/2 + caster_wheel_radius} 0 ${-chassis_height/2}" rpy="0 0 0"/>
+      <origin xyz="${caster_wheel_radius} 0 0" rpy="0 0 0"/>
     </joint>
     <!-- caster rear wheel Link -->
@@ -170,11 +156,11 @@
           iyy="${caster_wheel_mass * 0.4 * (caster_wheel_radius * caster_wheel_radius)}" iyz="0.0"
           izz="${caster_wheel_mass * 0.4 * (caster_wheel_radius * caster_wheel_radius)}"/>
-        </inertial>
-      </link>
+      </inertial>
+    </link>
     <!-- Hat joint -->
     <joint name="${prefix}hat_joint" type="fixed">
       <parent link="${prefix}chassis"/>
       <child link="${prefix}hat"/>
-      <origin xyz="0.03 0 ${chassis_height/2}" rpy="0 0 0"/>
+      <origin xyz="${chassis_length/2} 0 ${chassis_height}" rpy="0 0 0"/>
     </joint>
     <!-- Hat link -->

Commit message: parametrized the protobot_core macro so that sensors could be added using veriables instead of hardcoding

File: urdf/protobot.urdf.xacro (robot description, xacro)
@@ -7,18 +7,34 @@
     <!-- RVIZ colors -->
     <xacro:include filename="$(find protobot_description)/urdf/materials.urdf.xacro" />
+    <xacro:property name="chassis_length" value="0.3"/>
+    <xacro:property name="wheel_axis_horizontal_offset" value="${chassis_length - 0.02}"/>
+    <xacro:property name="wheel_axis_vertical_offset" value="0.04"/>
+    <xacro:property name="wheel_radius" value="0.06"/>
     <!-- Use macros from imported files to define the full protobot -->
-    <!--TODO: Parametrize the core macro so that camera and IMU can be placed without hardcoding -->
     <!-- Core URDF -->
     <xacro:include filename="$(find protobot_description)/urdf/protobot_core.urdf.xacro" />
-    <xacro:protobot_core prefix="$(arg prefix)"/>
+    <xacro:protobot_core prefix="$(arg prefix)"
+        chassis_mass="1.0"
+        chassis_length="${chassis_length}"
+        chassis_width="0.25"
+        chassis_height="0.15"
+        wheel_base="0.31"
+        wheel_mass="0.2"
+        wheel_width="0.030"
+        wheel_radius="${wheel_radius}"
+        wheel_axis_vertical_offset="${wheel_axis_vertical_offset}"
+        wheel_axis_horizontal_offset="${wheel_axis_horizontal_offset}"
+        caster_wheel_radius="${wheel_radius - wheel_axis_vertical_offset}"
+        caster_wheel_mass="0.1"
+    />
     <!-- Camera -->
     <xacro:include filename="$(find protobot_description)/urdf/camera.urdf.xacro" />
     <xacro:camera parent="chassis" prefix="$(arg prefix)">
-        <origin xyz="0.3 0 0.1" rpy="0 0 0" />
+        <origin xyz="${chassis_length} 0 0.1" rpy="0 0 0" />
     </xacro:camera>
     <!-- Inertial Measurement Unit (IMU) -->
     <xacro:include filename="$(find protobot_description)/urdf/imu_sensor.urdf.xacro" />
     <xacro:imu_sensor prefix="$(arg prefix)" parent="chassis">
-        <origin xyz="0.28 0 0.04" rpy="0 0 0" />
+        <origin xyz="${wheel_axis_horizontal_offset} 0 ${wheel_axis_vertical_offset}" rpy="0 0 0" />
     </xacro:imu_sensor>
     <!-- ROS2 Control -->

File: urdf/protobot_core.urdf.xacro (robot description, xacro)
@@ -2,34 +2,21 @@
 <robot xmlns:xacro="http://www.ros.org/wiki/xacro">
 <!-- Modified from: https://github.com/ros-controls/ros2_control_demos/blob/master/ros2_control_demo_description/diffbot/urdf/diffbot_description.urdf.xacro -->
-  <xacro:macro name="protobot_core" params="prefix">
-    <!-- TODO: Set these as macro parameters
-      prefix:=''
-      chassis_mass:='1.0'
-      chassis_length:='0.3'
-      chassis_width:='0.25'
-      chassis_height:='0.15'
-      wheel_base:='0.31'
-      wheel_mass:='0.2'
-      wheel_width:='0.030'
-      wheel_radius:='0.06'
-      wheel_axis_vertical_offset:='0.04'
-      wheel_axis_horizontal_offset:='0.28'
-      caster_wheel_radius:='0.02'
-      caster_wheel_mass:='0.1'
-  -->
+  <xacro:macro name="protobot_core" params="prefix
+    chassis_mass:=1.0
+    chassis_length:=0.3
+    chassis_width:=0.25
+    chassis_height:=0.15
+    wheel_base:=0.31
+    wheel_mass:=0.2
+    wheel_width:=0.030
+    wheel_radius:=0.06
+    wheel_axis_vertical_offset:=0.04
+    wheel_axis_horizontal_offset:=0.28
+    caster_wheel_radius:=0.02
+    caster_wheel_mass:=0.1">
+    <!-- to keep the robot horizontal, set:
+      caster_wheel_radius = wheel_radius - wheel_axis_vertical_offset-->
     <!-- Constants for robot dimensions -->
     <xacro:property name="PI" value="3.1415926535897931"/>
-    <xacro:property name="chassis_mass" value="1.0" /> <!-- arbitrary value for base mass -->
-    <xacro:property name="chassis_length" value="0.3" />
-    <xacro:property name="chassis_width" value="0.25" />
-    <xacro:property name="chassis_height" value="0.3" />
-    <xacro:property name="wheel_base" value="0.31" /> <!-- make this bigger than chassis_width -->
-    <xacro:property name="wheel_mass" value="0.2" /> <!-- arbitrary value for wheel mass -->
-    <xacro:property name="wheel_width" value="0.030" />
-    <xacro:property name="wheel_radius" value="0.06" />
-    <xacro:property name="wheel_axis_vertical_offset" value="0.04" /> <!-- signed vertical distance from bottom of chassis to wheel axis -->
-    <xacro:property  name="wheel_axis_horizontal_offset" value="${chassis_length - 0.02}" /> <!-- signed horizontal distance from back of chassis to wheel axis -->
-    <xacro:property name="caster_wheel_mass" value="0.1" /> <!-- arbitrary value for caster wheel mass -->
-    <xacro:property name="caster_wheel_radius" value="${wheel_radius - wheel_axis_vertical_offset}" />
     <!-- Dummy link with no inertiais used as root (for gazebo) -->
     <link name="base_link"/>

Commit message: changed wheels to be wrt base_link

File: urdf/protobot.urdf.xacro (robot description, xacro)
@@ -8,6 +8,6 @@
     <xacro:include filename="$(find protobot_description)/urdf/materials.urdf.xacro" />
     <xacro:property name="chassis_length" value="0.3"/>
-    <xacro:property name="wheel_axis_horizontal_offset" value="${chassis_length - 0.02}"/>
-    <xacro:property name="wheel_axis_vertical_offset" value="0.04"/>
+    <xacro:property name="wheel_axis_wrt_chassis_horizontal" value="${chassis_length - 0.02}"/>
+    <xacro:property name="wheel_axis_wrt_chassis_vertical" value="0.04"/>
     <xacro:property name="wheel_radius" value="0.06"/>
     <!-- Use macros from imported files to define the full protobot -->
@@ -23,7 +23,7 @@
         wheel_width="0.020"
         wheel_radius="${wheel_radius}"
-        wheel_axis_vertical_offset="${wheel_axis_vertical_offset}"
-        wheel_axis_horizontal_offset="${wheel_axis_horizontal_offset}"
-        caster_wheel_radius="${wheel_radius - wheel_axis_vertical_offset}"
+        wheel_axis_wrt_chassis_vertical="${wheel_axis_wrt_chassis_vertical}"
+        wheel_axis_wrt_chassis_horizontal="${wheel_axis_wrt_chassis_horizontal}"
+        caster_wheel_radius="${wheel_radius - wheel_axis_wrt_chassis_vertical}"
         caster_wheel_mass="0.1"
     />
@@ -36,5 +36,5 @@
     <xacro:include filename="$(find protobot_description)/urdf/imu_sensor.urdf.xacro" />
     <xacro:imu_sensor prefix="$(arg prefix)" parent="chassis" use_gazebo="$(arg use_gazebo)">
-        <origin xyz="${wheel_axis_horizontal_offset} 0 ${wheel_axis_vertical_offset}" rpy="0 0 0" />
+        <origin xyz="${wheel_axis_wrt_chassis_horizontal} 0 ${wheel_axis_wrt_chassis_vertical}" rpy="0 0 0" />
     </xacro:imu_sensor>
     <!-- ROS2 Control -->

File: urdf/protobot_core.urdf.xacro (robot description, xacro)
@@ -11,14 +11,22 @@
     wheel_width:=0.030
     wheel_radius:=0.06
-    wheel_axis_vertical_offset:=0.04
-    wheel_axis_horizontal_offset:=0.28
+    wheel_axis_wrt_chassis_vertical:=0.04
+    wheel_axis_wrt_chassis_horizontal:=0.28
     caster_wheel_radius:=0.02
     caster_wheel_mass:=0.1">
     <!-- to keep the robot horizontal, set:
-      caster_wheel_radius = wheel_radius - wheel_axis_vertical_offset-->
+      caster_wheel_radius = wheel_radius - wheel_axis_wrt_chassis_vertical-->
     <!-- Constants for robot dimensions -->
     <xacro:property name="PI" value="3.1415926535897931"/>
-    <!-- Dummy link with no inertiais used as root (for gazebo) -->
+    <!-- Frame at the midpoint of the wheel axis serves a the pendulum pivot point, and has no inertial properties for gazebo. -->
     <link name="base_link"/>
+    <!-- Coordinate frame that is analogous to the mass of the pendulum.
+    It is located at the robot's center of mass, and the x-axis intersects the base_link. -->
+    <!-- <link name="${prefix}pendulum_mass"/> -->
+    <!-- <joint name="${prefix}pendulum_mass_joint" type="fixed">
+      <parent link="base_link"/>
+      <child link="${prefix}pendulum_mass"/>
+      <origin xyz="${-wheel_axis_wrt_chassis_horizontal+chassis_length/2} 0 ${-wheel_axis_wrt_chassis_vertical+chassis_height/2}" rpy="0 ${PI/2} 0"/>
+    </joint> -->
     <!-- Chassis Link -->
     <link name="${prefix}chassis">
@@ -48,10 +56,10 @@
       <parent link="base_link"/>
       <child link="${prefix}chassis"/>
-      <origin xyz="${-wheel_axis_horizontal_offset} 0 ${-wheel_axis_vertical_offset}" rpy="0 0 0" />
+      <origin xyz="${-wheel_axis_wrt_chassis_horizontal} 0 ${-wheel_axis_wrt_chassis_vertical}" rpy="0 0 0" />
     </joint>
     <joint name="${prefix}left_wheel_joint" type="continuous">
-      <parent link="${prefix}chassis"/>
+      <parent link="${prefix}base_link"/>
       <child link="${prefix}left_wheel"/>
-      <origin xyz="${wheel_axis_horizontal_offset} ${wheel_base/2} ${wheel_axis_vertical_offset}" rpy="${-PI/2} 0 0"/>
+      <origin xyz="0 ${wheel_base/2} 0" rpy="${-PI/2} 0 0"/>
       <axis xyz="0 0 1"/>
       <!-- <dynamics damping="0.2"/>
@@ -84,7 +92,7 @@
     </link>
     <joint name="${prefix}right_wheel_joint" type="continuous">
-      <parent link="${prefix}chassis"/>
+      <parent link="${prefix}base_link"/>
       <child link="${prefix}right_wheel"/>
-      <origin xyz="${wheel_axis_horizontal_offset} ${-wheel_base/2} ${wheel_axis_vertical_offset}" rpy="${PI/2} 0 0"/>
+      <origin xyz="0 ${-wheel_base/2} 0" rpy="${PI/2} 0 0"/>
       <axis xyz="0 0 -1"/> <!-- Note that "Forward" rotation is opposite compared to the left wheel -->
       <!-- <dynamics damping="0.2"/>
