Commit message: remove front caster wheel and move wheels forward

File: urdf/protobot_core.urdf.xacro (robot description, xacro)
@@ -5,13 +5,14 @@
   <!-- Constants for robot dimensions -->
   <xacro:property name="PI" value="3.1415926535897931"/>
-  <xacro:property name="chassis_mass" value="0.5" /> <!-- arbitrary value for base mass -->
+  <xacro:property name="chassis_mass" value="1.0" /> <!-- arbitrary value for base mass -->
   <xacro:property name="chassis_length" value="0.3" />
   <xacro:property name="chassis_width" value="0.25" />
   <xacro:property name="chassis_height" value="0.15" />
   <xacro:property name="wheel_base" value="0.31" /> <!-- make this bigger than chassis_width -->
-  <xacro:property name="wheel_mass" value="0.3" /> <!-- arbitrary value for wheel mass -->
+  <xacro:property name="wheel_mass" value="0.2" /> <!-- arbitrary value for wheel mass -->
   <xacro:property name="wheel_width" value="0.030" />
-  <xacro:property name="wheel_radius" value="0.05" />
-  <xacro:property name="wheel_axis_vertical_offset" value="-0.04" /> <!-- signed distance from chassis center to wheel axis -->
+  <xacro:property name="wheel_radius" value="0.06" />
+  <xacro:property name="wheel_axis_vertical_offset" value="-0.04" /> <!-- signed vertical distance from chassis center to wheel axis -->
+  <xacro:property  name="wheel_axis_horizontal_offset" value="${chassis_length/2 - 0.02}" /> <!-- signed horizontal distance from chassis center to wheel axis -->
   <xacro:property name="caster_wheel_mass" value="0.1" /> <!-- arbitrary value for caster wheel mass -->
   <xacro:property name="caster_wheel_radius" value="${-wheel_axis_vertical_offset + wheel_radius - chassis_height/2}" />
@@ -50,5 +51,5 @@
       <parent link="${prefix}chassis"/>
       <child link="${prefix}left_wheel"/>
-      <origin xyz="0 ${chassis_length/2} ${wheel_axis_vertical_offset}" rpy="${-PI/2} 0 0"/>
+      <origin xyz="${wheel_axis_horizontal_offset} ${chassis_length/2} ${wheel_axis_vertical_offset}" rpy="${-PI/2} 0 0"/>
       <axis xyz="0 0 1"/>
       <!-- <dynamics damping="0.2"/>
@@ -83,5 +84,5 @@
       <parent link="${prefix}chassis"/>
       <child link="${prefix}right_wheel"/>
-      <origin xyz="0 ${-chassis_length/2} ${wheel_axis_vertical_offset}" rpy="${PI/2} 0 0"/>
+      <origin xyz="${wheel_axis_horizontal_offset} ${-chassis_length/2} ${wheel_axis_vertical_offset}" rpy="${PI/2} 0 0"/>
       <axis xyz="0 0 -1"/> <!-- Note that "Forward" rotation is opposite compared to the left wheel -->
       <!-- <dynamics damping="0.2"/>
@@ -113,11 +114,11 @@
         </inertial>
       </link>
-    <joint name="${prefix}front_caster_wheel_joint" type="fixed">
+    <!-- <joint name="${prefix}front_caster_wheel_joint" type="fixed">
       <parent link="${prefix}chassis"/>
       <child link="${prefix}front_caster_wheel"/>
       <origin xyz="${chassis_length/2 - caster_wheel_radius} 0 ${-chassis_height/2}" rpy="0 0 0"/>
-    </joint>
+    </joint> -->
     <!-- caster front wheel Link -->
-    <link name="${prefix}front_caster_wheel">
+    <!-- <link name="${prefix}front_caster_wheel">
       <collision>
         <origin xyz="0 0 0" rpy="0 0 0"/>
@@ -141,5 +142,5 @@
           izz="${caster_wheel_mass * 0.4 * (caster_wheel_radius * caster_wheel_radius)}"/>
         </inertial>
-      </link>
+      </link> -->
     <joint name="${prefix}rear_caster_wheel_joint" type="fixed">
       <parent link="${prefix}chassis"/>

Commit message: protobot_gazebo reference names need to match protobot_core

File: urdf/protobot_core.urdf.xacro (robot description, xacro)
@@ -116,11 +116,11 @@
       </inertial>
     </link>
-    <joint name="${prefix}rear_caster_wheel_joint" type="fixed">
+    <joint name="${prefix}caster_wheel_joint" type="fixed">
       <parent link="${prefix}chassis"/>
-      <child link="${prefix}rear_caster_wheel"/>
+      <child link="${prefix}caster_wheel"/>
       <origin xyz="${caster_wheel_radius} 0 0" rpy="0 0 0"/>
     </joint>
     <!-- caster rear wheel Link -->
-    <link name="${prefix}rear_caster_wheel">
+    <link name="${prefix}caster_wheel">
       <collision>
         <origin xyz="0 0 0" rpy="0 0 0"/>

File: urdf/protobot_gazebo.urdf.xacro (robot description, xacro)
@@ -4,26 +4,25 @@
   <xacro:macro name="protobot_gazebo" params="prefix">
     <!-- Define the friction and colors to use in simulation (Gazebo is unable to use the same <material> tags as the URDF) -->
-    <gazebo reference="chassis_link">
+    <gazebo reference="${prefix}chassis">
         <material>Gazebo/Blue</material>
     </gazebo>
-    <gazebo reference="left_wheel">
-        <mu1>0.8</mu1> <!-- contact friction: rubber on dry asphalt -->
-        <mu2>0.8</mu2>
-        <material>Gazebo/Black</material>
+    <gazebo reference="${prefix}left_wheel">
+        <mu1>1.0</mu1> <!-- contact friction -->
+        <mu2>1.0</mu2>
+        <kp>1e10</kp> <!-- stiffness -->
+        <kd>1e10</kd> <!-- damping -->
+        <material>Gazebo/Red</material>
     </gazebo>
-    <gazebo reference="right_wheel">
-        <mu1>0.8</mu1> <!-- contact friction: rubber on dry asphalt -->
-        <mu2>0.8</mu2>
-        <material>Gazebo/Black</material>
+    <gazebo reference="${prefix}right_wheel">
+        <mu1>1.0</mu1> <!-- contact friction -->
+        <mu2>1.0</mu2>
+        <kp>1e10</kp> <!-- stiffness -->
+        <kd>1e10</kd> <!-- damping -->
+        <material>Gazebo/Red</material>
     </gazebo>
-    <gazebo reference="front_caster_wheel">
-        <mu1>0.001</mu1> <!-- contact friction coefficient -->
-        <mu2>0.001</mu2>
-        <material>Gazebo/Black</material>
-    </gazebo>
-    <gazebo reference="rear_caster_wheel">
-        <mu1>0.001</mu1> <!-- contact friction coefficient -->
-        <mu2>0.001</mu2>
-        <material>Gazebo/Black</material>
+    <gazebo reference="${prefix}caster_wheel">
+        <mu1>0.000001</mu1> <!-- contact friction coefficient -->
+        <mu2>0.000001</mu2>
+        <material>Gazebo/Red</material>
     </gazebo>
     <!-- ros2 control plugin -->

Commit message: added pendulum_mass frame (and use pi instead of PI)

File: urdf/protobot_core.urdf.xacro (robot description, xacro)
@@ -17,16 +17,16 @@
     <!-- to keep the robot horizontal, set:
       caster_wheel_radius = wheel_radius - wheel_axis_wrt_chassis_vertical-->
-    <!-- Constants for robot dimensions -->
-    <xacro:property name="PI" value="3.1415926535897931"/>
     <!-- Frame at the midpoint of the wheel axis serves a the pendulum pivot point, and has no inertial properties for gazebo. -->
     <link name="base_link"/>
     <!-- Coordinate frame that is analogous to the mass of the pendulum.
     It is located at the robot's center of mass, and the x-axis intersects the base_link. -->
-    <!-- <link name="${prefix}pendulum_mass"/> -->
-    <!-- <joint name="${prefix}pendulum_mass_joint" type="fixed">
+    <link name="${prefix}pendulum_mass"/>
+    <joint name="${prefix}pendulum_mass_joint" type="fixed">
       <parent link="base_link"/>
       <child link="${prefix}pendulum_mass"/>
-      <origin xyz="${-wheel_axis_wrt_chassis_horizontal+chassis_length/2} 0 ${-wheel_axis_wrt_chassis_vertical+chassis_height/2}" rpy="0 ${PI/2} 0"/>
-    </joint> -->
+      <origin
+        xyz="${-wheel_axis_wrt_chassis_horizontal+chassis_length/2} 0 ${-wheel_axis_wrt_chassis_vertical+chassis_height/2}"
+        rpy="0 ${atan2(-wheel_axis_wrt_chassis_vertical+chassis_height/2, -(-wheel_axis_wrt_chassis_horizontal+chassis_length/2))} 0"/>
+    </joint>
     <!-- Chassis Link -->
     <link name="${prefix}chassis">
@@ -61,5 +61,5 @@
       <parent link="${prefix}base_link"/>
       <child link="${prefix}left_wheel"/>
-      <origin xyz="0 ${wheel_base/2} 0" rpy="${-PI/2} 0 0"/>
+      <origin xyz="0 ${wheel_base/2} 0" rpy="${-pi/2} 0 0"/>
       <axis xyz="0 0 1"/>
       <!-- <dynamics damping="0.2"/>
@@ -94,5 +94,5 @@
       <parent link="${prefix}base_link"/>
       <child link="${prefix}right_wheel"/>
-      <origin xyz="0 ${-wheel_base/2} 0" rpy="${PI/2} 0 0"/>
+      <origin xyz="0 ${-wheel_base/2} 0" rpy="${pi/2} 0 0"/>
       <axis xyz="0 0 -1"/> <!-- Note that "Forward" rotation is opposite compared to the left wheel -->
       <!-- <dynamics damping="0.2"/>

Commit message: z-axis intersects base_link, not x-axis

File: urdf/protobot_core.urdf.xacro (robot description, xacro)
@@ -20,12 +20,14 @@
     <link name="base_link"/>
     <!-- Coordinate frame that is analogous to the mass of the pendulum.
-    It is located at the robot's center of mass, and the x-axis intersects the base_link. -->
+    It is located at the robot's center of mass, and the z-axis intersects the base_link. -->
     <link name="${prefix}pendulum_mass"/>
+    <xacro:property name="mass_center_z" value="${-wheel_axis_wrt_chassis_vertical+chassis_height/2}"/>
+    <xacro:property name="mass_center_x" value="${-wheel_axis_wrt_chassis_horizontal+chassis_length/2}"/>
     <joint name="${prefix}pendulum_mass_joint" type="fixed">
       <parent link="base_link"/>
       <child link="${prefix}pendulum_mass"/>
       <origin
-        xyz="${-wheel_axis_wrt_chassis_horizontal+chassis_length/2} 0 ${-wheel_axis_wrt_chassis_vertical+chassis_height/2}"
-        rpy="0 ${atan2(-wheel_axis_wrt_chassis_vertical+chassis_height/2, -(-wheel_axis_wrt_chassis_horizontal+chassis_length/2))} 0"/>
+        xyz="${mass_center_x} 0 ${mass_center_z}"
+        rpy="0 ${-atan2(-mass_center_x, mass_center_z)} 0"/>
     </joint>
     <!-- Chassis Link -->

Commit message: pendulum_frame instead of pendulum_mass

File: urdf/protobot_core.urdf.xacro (robot description, xacro)
@@ -20,11 +20,11 @@
     <link name="base_link"/>
     <!-- Coordinate frame that is analogous to the mass of the pendulum.
-    It is located at the robot's center of mass, and the z-axis intersects the base_link. -->
-    <link name="${prefix}pendulum_mass"/>
+    It is located at the robot's center of mass, and the z-axis intersects the base_link such that zero pitch is balanced. -->
+    <link name="${prefix}pendulum_frame"/>
     <xacro:property name="mass_center_z" value="${-wheel_axis_wrt_chassis_vertical+chassis_height/2}"/>
     <xacro:property name="mass_center_x" value="${-wheel_axis_wrt_chassis_horizontal+chassis_length/2}"/>
-    <joint name="${prefix}pendulum_mass_joint" type="fixed">
+    <joint name="${prefix}pendulum_frame_joint" type="fixed">
       <parent link="base_link"/>
-      <child link="${prefix}pendulum_mass"/>
+      <child link="${prefix}pendulum_frame"/>
       <origin
         xyz="${mass_center_x} 0 ${mass_center_z}"
